File: letitrain.kicad_pcb (KiCad board)
At the start: 2 copper layers, 71 x 51 mm, 47 parts, among them J1 Conn_01x05, J2 Conn_01x05, J3 Conn_01x03, J4 Screw_Terminal_01x02, J5 Conn_01x04, J6 Conn_01x03_Pin, J7 Screw_Terminal_01x02, J8 Conn_01x02, J9 Conn_01x02, Q1 BSS84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

Commit message: Update to v1.1
Parts:
- U1: value MCP9701 -> MCP9700B; footprint Package_TO_SOT_SMD:SOT-353_SC-70-5 -> Package_TO_SOT_SMD:SOT-23_Handsoldering
- moved J6 2.40 mm to (73.4, 66.0)
- moved C8 2.40 mm to (73.0, 62.6)
- moved C9 2.40 mm to (68.8, 62.6)
- moved J8 0.77 mm to (64.2, 60.6)
- moved J9 0.77 mm to (64.2, 64.8)
- moved U1 0.47 mm to (34.7, 52.5)
- turned D1 to 180 degrees
Connections:
- D1 pad 1: GND -> +12V
- D1 pad 2: +12V -> GND
- U1 pad 1: unconnected-(U1-NC-Pad1) -> +3V3
- U1 pad 2: GND -> /ADC_TEMP
- U1 pad 3: /ADC_TEMP -> GND
Routing:
- net +12V: track 58.0 -> 60.4 mm
- net +3V3: track 102.6 -> 104.5 mm
- net GND: track 13.9 -> 12.5 mm
- net /ADC_TEMP: track 10.9 -> 10.3 mm
Other:
- board text added: "v1.1"
- board text removed: "v1"
