File: letitrain.kicad_sch (KiCad schematic)
At the start: 33 parts, among them J1 Conn_01x05, J2 Conn_01x05, J3 Conn_01x03, J5 Conn_01x04, J6 Conn_01x03_Pin, J7 Screw_Terminal_01x02, J8 Conn_01x02, J9 Conn_01x02, U1 MCP9701, U2 ESP32-WROOM-32D

Commit message: Update to v1.1
Parts:
- C9: symbol Device:C_Polarized -> Device:C
- D1, J1, J2, J5, J8, J9, R16: now not fitted
- U1: value MCP9701 -> MCP9700B; footprint Package_TO_SOT_SMD:SOT-353_SC-70-5 -> Package_TO_SOT_SMD:SOT-23_Handsoldering; now not fitted
Connections:
- net +12V: now also D1.1 (A1); no longer D1.2 (A2)
- net +3V3: now also U1.1 (V_{DD}); no longer U1.4 (V_{DD})
- net ADC_TEMP: now also U1.2 (V_{OUT}); no longer U1.3 (V_{OUT})
- net GND: now also D1.2 (A2), U1.3 (GND); no longer D1.1 (A1), U1.2 (GND)
Changed lines of the file:
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@@
 		(in_bom yes)
 		(on_board yes)
-		(dnp no)
+		(dnp yes)
 		(fields_autoplaced yes)
 		(property "Reference" "J2"
@@
 		(in_bom yes)
 		(on_board yes)
-		(dnp no)
+		(dnp yes)
 		(fields_autoplaced yes)
 		(property "Reference" "R16"
@@
 		(in_bom yes)
 		(on_board yes)
-		(dnp no)
+		(dnp yes)
 		(fields_autoplaced yes)
 		(property "Reference" "J8"
@@
 		(in_bom yes)
 		(on_board yes)
-		(dnp no)
+		(dnp yes)
 		(fields_autoplaced yes)
 		(property "Reference" "U1"
@@
 			)
 		)
-		(property "Value" "MCP9701"
+		(property "Value" "MCP9700B"
 			(at 85.09 125.7299 0)
 			(effects
@@
 			)
 		)
-		(property "Footprint" "Package_TO_SOT_SMD:SOT-353_SC-70-5"
+		(property "Footprint" "Package_TO_SOT_SMD:SOT-23_Handsoldering"
 			(at 93.98 134.62 0)
 			(effects
@@
 			)
 		)
-		(pin "5"
-		)
 		(pin "1"
 		)
 		(pin "3"
 		)
-		(pin "4"
-		)
 		(pin "2"
 		)
@@
 		(in_bom yes)
 		(on_board yes)
-		(dnp no)
+		(dnp yes)
 		(fields_autoplaced yes)
 		(property "Reference" "J5"
@@
 	)
 	(symbol
-		(lib_id "Device:C_Polarized")
+		(lib_id "Device:C")
 		(at 99.06 177.8 0)
 		(unit 1)
@@
 		(fields_autoplaced yes)
 		(property "Reference" "C9"
-			(at 102.87 175.6409 0)
+			(at 102.87 176.5299 0)
 			(effects
 				(font
@@
 		)
 		(property "Value" "10u"
-			(at 102.87 178.1809 0)
+			(at 102.87 179.0699 0)
 			(effects
 				(font
@@
 			)
 		)
-		(property "Description" "Polarized capacitor"
+		(property "Description" "Unpolarized capacitor"
 			(at 99.06 177.8 0)
 			(effects
@@
 		(in_bom yes)
 		(on_board yes)
-		(dnp no)
+		(dnp yes)
 		(fields_autoplaced yes)
 		(property "Reference" "J9"
@@
 	(symbol
 		(lib_id "Device:D_TVS")
-		(at 64.77 76.2 90)
+		(at 64.77 76.2 270)
 		(unit 1)
 		(exclude_from_sim no)
 		(in_bom yes)
 		(on_board yes)
-		(dnp no)
+		(dnp yes)
 		(property "Reference" "D1"
-			(at 67.31 74.9299 90)
+			(at 62.23 77.4701 90)
 			(effects
 				(font
@@
 		)
 		(property "Value" "P4SMAJ30CA"
-			(at 67.31 77.4699 90)
+			(at 62.23 74.9301 90)
 			(effects
 				(font
@@
 		(in_bom yes)
 		(on_board yes)
-		(dnp no)
+		(dnp yes)
 		(fields_autoplaced yes)
 		(property "Reference" "J1"
